Commit message: update hand_rotation

File: LeapHand_rotation/assets/urdf/leap_hand_xarm/leap_hand_change.urdf (robot description, URDF)
Before this commit: robot xarm6_leap_hand_with_fsr, 41 links, 40 joints
Links:
- link onshape_thumb_fingertip: geometry collision mesh filename=meshes/long_thin_thumbtip_2.obj scale=1. 1. 1.; visual mesh filename=meshes/long_thin_thumbtip_2.obj scale=1. 1. 1.
Joints:
- joint thumb_tip: origin xyz=0.0102383 -0.0453895 0.0144321 rpy=3.1415927 0. 0.0000001 -> xyz=0.0020383 -0.0600895 0.0144321 rpy=3.1415927 0. 0.0000001

File: LeapHand_rotation/assets/urdf/leap_hand_xarm/meshes/leap_hand_change.urdf (robot description, URDF)
Before this commit: robot xarm6_leap_hand_with_fsr, 41 links, 40 joints
Links:
- link dip_1_fsr: geometry collision mesh filename=meshes/dip_1_fsr_Cube.obj scale=0.5 0.8 0.5; visual mesh filename=meshes/dip_1_fsr_Cube.obj scale=0.5 0.8 0.5
- link dip_2_fsr: geometry collision mesh filename=meshes/dip_2_fsr_Cube.obj scale=0.5 0.8 0.5; visual mesh filename=meshes/dip_2_fsr_Cube.obj scale=0.5 0.8 0.5
- link dip_3_fsr: geometry collision mesh filename=meshes/dip_3_fsr_Cube.obj scale=0.5 0.8 0.5; visual mesh filename=meshes/dip_3_fsr_Cube.obj scale=0.5 0.8 0.5
- link onshape_thumb_fingertip: geometry collision mesh filename=meshes/thin_thumbtip.obj scale=1. 1. 1.; visual mesh filename=meshes/thin_thumbtip.obj scale=1. 1. 1.
- link thumb_dip_fsr: geometry collision mesh filename=meshes/thumb_dip_fsr_Cube.obj scale=1. 0.5 1.; visual mesh filename=meshes/thumb_dip_fsr_Cube.obj scale=1. 0.5 1.
- link thumb_pip_fsr: geometry collision mesh filename=meshes/thumb_pip_fsr_Cube.obj scale=1. 0.5 1.; visual mesh filename=meshes/thumb_pip_fsr_Cube.obj scale=1. 0.5 1.
Joints:
- joint dip_1: origin xyz=0.0084151 -0.0367202 -0.0143087 rpy=1.5707964 -0. -1.5707964 -> xyz=0.0090151 -0.0227202 -0.0143087 rpy=1.5707964 -0. -1.5707964
- joint dip_2_fsr_dip_2: origin xyz=0.0084151 -0.0367202 -0.0147031 rpy=1.5707964 -0.0000001 -1.5707964 -> xyz=0.0090151 -0.0227202 -0.0147031 rpy=1.5707964 -0.0000001 -1.5707964
- joint dip_3_fsr_dip_3: origin xyz=0.0084151 -0.0367202 -0.0145862 rpy=1.5707964 -0.0000001 -1.5707964 -> xyz=0.0090151 -0.0227202 -0.0145862 rpy=1.5707964 -0.0000001 -1.5707964
- joint pip_1: origin xyz=0.0020601 -0.0000087 0.0230151 rpy=3.1415925 0. 3.1415925 -> xyz=0.0019601 -0.0000087 0.0230151 rpy=3.1415925 0. 3.1415925
- joint pip_2_fsr_pip_2: origin xyz=0.0020601 -0.0002805 0.0230151 rpy=3.1415925 0. 3.1415925 -> xyz=0.0019601 -0.0002805 0.0230151 rpy=3.1415925 0. 3.1415925
- joint pip_3_fsr_pip_3: origin xyz=0.0020601 0.0007753 0.0230151 rpy=3.1415925 0. 3.1415925 -> xyz=0.0019601 0.0007753 0.0230151 rpy=3.1415925 0. 3.1415925
- joint thumb_dip_fsr_thumb_dip: origin xyz=0.0094383 -0.007675 0.0144321 rpy=3.1415927 0. 0.0000001 -> xyz=0.0094383 -0.017675 0.0144321 rpy=3.1415927 0. 0.0000001
- joint thumb_pip_fsr_thumb_pip: origin xyz=-0.0094383 0.0105035 0.0142321 rpy=3.1415925 0. -3.1415927 -> xyz=-0.0094383 0.0205035 0.0142321 rpy=3.1415925 0. -3.1415927
- joint thumb_tip: origin xyz=0.0102383 -0.0453895 0.0144321 rpy=3.1415927 0. 0.0000001 -> xyz=0.0020383 -0.0600895 0.0144321 rpy=3.1415927 0. 0.0000001
